File: wrist_watch/programmer/programmer.kicad_pcb (KiCad board)
At the start: 2 copper layers, 59.9 x 46.7 mm, 47 parts, among them J1 Conn_01x01, J10 Conn_01x01, J11 Conn_01x01, J12 Conn_01x01, J13 Conn_02x03_Counter_Clockwise, J14 USB_C_Receptacle_USB2.0_MPN, J15 Conn_02x03_Counter_Clockwise, J2 Conn_01x01, J3 Conn_01x01, J4 Conn_01x01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

Commit message: silkscreen update
Parts:
- added kibuzzard-67CEF9E0: G***, kibuzzard-67CEF9E0, F.Cu at (127.5, 113.5)
